File: hardware/electronics/main_board/main_board.sch (KiCad schematic (older format))
At the start: 89 parts, among them J1 Conn_01x04_Female, Q1 CSD18537NQ5A, Q2 CSD18537NQ5A, Q3 CSD18537NQ5A, Q4 CSD18537NQ5A

Commit message: pcb looking much better
Parts:
- removed C_12v_0, C_3.3v_0: 220uF, Capacitor_SMD:C_Elec_10x10.2, symbol Device:CP
- removed C_tmc_6: 2.2u, Capacitor_SMD:C_0603_1608Metric, symbol Device:C_Small
- removed C_tmc_7: 100nF, symbol Device:C_Small
- removed J1: Conn_01x04_Female, Connector_Molex:Molex_Nano-Fit_105310-xx04_2x02_P2.50mm_Vertical, symbol Connector:Conn_01x04_Female
- removed PROG1, RESET1: SW_Push_Dual, Button_Switch_SMD:SW_Push_1P1T_NO_6x6mm_H9.5mm, symbol Switch:SW_Push_Dual
- added C1: 10uF, Capacitor_SMD:C_0402_1005Metric, symbol Device:C
- added C2: 100nF, Capacitor_SMD:C_0402_1005Metric, symbol Device:C_Small
- added C_12v_?, C_3.3v_?: 220uF, Capacitor_SMD:C_Elec_10x10.2, symbol Device:C
- added C_TMC_28, C_TMC_29: 1n, Capacitor_SMD:C_1206_3216Metric, symbol Device:C_Small
- added C_esp_1, C_esp_2: 100pF, Capacitor_SMD:C_0603_1608Metric, symbol Device:C_Small
- added C_tmc_10: 220nF, Capacitor_SMD:C_1206_3216Metric, symbol Device:C_Small
- added C_tmc_11, C_tmc_?: 2.2u, Capacitor_SMD:C_1206_3216Metric, symbol Device:C_Small
- added C_tmc_13, C_tmc_15: 4.7uF, Capacitor_SMD:C_1206_3216Metric, symbol Device:C_Small
- added C_tmc_14, C_tmc_? (x2): 100nF, Capacitor_SMD:C_1206_3216Metric, symbol Device:C_Small
- added D1: LED, LED_SMD:LED_0603_1608Metric, symbol Device:LED
- added D_1esp_1, D_1esp_2, D_tmc_2, D_tmc_4: STPS3L60U, Diode_SMD:D_2114_3652Metric, symbol Device:D_Schottky_Small
- added GPIO_EXP_1, GPIO_EXP_2, POWER_EXP_1: Conn_01x04_Male, Connector_PinHeader_2.54mm:PinHeader_1x04_P2.54mm_Vertical, symbol Connector:Conn_01x04_Male
- added J1: RJ45, main_board:2158771, symbol Connector:RJ45
- added J2: TF-15X15, main_board:TF15X15, symbol TF-15X15:TF-15X15
- added J3: Conn_02x04_Odd_Even, Connector_Molex:Molex_Micro-Fit_3.0_43045-0812_2x04_P3.00mm_Vertical, symbol Connector_Generic:Conn_02x04_Odd_Even
- added L12v_1: 47uH, Inductor_SMD:L_0805_2012Metric, symbol Device:L_Small
- added L_3.3_1: 100uH, Inductor_SMD:L_0805_2012Metric, symbol Device:L_Small
- added PROG1, RESET1: SW_Push_Dual_x2, Button_Switch_SMD:SW_Push_1P1T_NO_6x6mm_H9.5mm, symbol Switch:SW_Push_Dual_x2
- added Q5, Q6, Q7, Q8: CSD18537NQ5A, Package_TO_SOT_SMD:TDSON-8-1, symbol Transistor_FET:CSD18537NQ5A
- added R1: 300 Ohms, Resistor_SMD:R_0805_2012Metric, symbol Device:R_Small_US
- added R_TMC_1, R_TMC_2: 10kOhms, Resistor_SMD:R_1206_3216Metric, symbol Device:R_US
- added R_esp_1, R_esp_2, R_tmc_?: 1Ohm, Resistor_SMD:R_1206_3216Metric, symbol Device:R_Small_US
- added R_esp_3, R_esp_4: 750Ohm, Resistor_SMD:R_1206_3216Metric, symbol Device:R_Small_US
- added R_tmc_11, R_tmc_12, R_tmc_13, R_tmc_16, R_tmc_17, R_tmc_18, R_tmc_19: 10Ohm, Resistor_SMD:R_1206_3216Metric, symbol Device:R_Small_US
- added R_tmc_14, R_tmc_15: 47R, Resistor_SMD:R_0805_2012Metric, symbol Device:R_Small_US
- added U1: P82B96, Package_SO:SO-8_3.9x4.9mm_P1.27mm, symbol Interface_Expansion:P82B96
- C4: footprint (none) -> Capacitor_SMD:C_0402_1005Metric
- C_12_4, C_3.3_4: footprint (none) -> Capacitor_SMD:C_0805_2012Metric
- C_TMC_14: value 100nF -> 220nF; footprint Capacitor_SMD:C_1206_3216Metric -> Capacitor_SMD:C_0805_2012Metric; JLCPCB C24497 -> C5378
- C_tmc_8: value 4.7uF -> 470nF; JLCPCB C29823 -> C13967
- C_tmc_9: value 100nF -> 220nF; footprint (none) -> Capacitor_SMD:C_1206_3216Metric; JLCPCB C1525 -> C1857
- J_48v_IN1: value XT-30 -> Molex; footprint main_board:XT30PW-M -> Connector_Molex:Molex_Micro-Fit_3.0_43045-0212_2x01_P3.00mm_Vertical; JLCPCB (none) -> C293362
- L3.3_1: value 126uH -> 47uH; footprint Inductor_SMD:L_0402_1005Metric -> Inductor_SMD:L_0805_2012Metric; JLCPCB (none) -> C14304; JLPCB C77120 -> (none)
- L_12v_1: value 126uH -> 100uH; footprint Inductor_SMD:L_0402_1005Metric -> Inductor_SMD:L_0805_2012Metric; JLCPCB (none) -> C68035; JLPCB C77120 -> (none)
- PHeader1: footprint Connector_Molex:Molex_PicoBlade_53047-0410_1x04_P1.25mm_Vertical -> Connector_PinHeader_2.54mm:PinHeader_1x04_P2.54mm_Vertical; JLCPCB C31597 -> C124378
- R_12v_2, R_3.3_2: footprint (none) -> Resistor_SMD:R_0805_2012Metric
- R_tmc_1: footprint (none) -> Resistor_SMD:R_0805_2012Metric; JLCPCB (none) -> C17521
- gave numbers to parts that had none: 2
Connections:
- net +12V: now also L_12v_1.1, J1.6, POWER_EXP_1.2 (Pin_2), R_esp_3.2, R_esp_4.1, U1.8 (VCC); no longer L_12v_1.2
- net +3V3: now also U_TRINAMIC1.11 (TST_MODE), U_TRINAMIC1.22 (SPI_MODE), C1.1, C1.2, C2.1, C2.2, C_TMC_28.1, C_TMC_29.1, C_esp_1.1, C_esp_2.2, C_tmc_13.2, C_tmc_14.2, C_tmc_15.2, C_tmc_?.2, C_tmc_?.2, D_1esp_1.2 (A), D_1esp_2.2 (A), D_tmc_2.2 (A), D_tmc_4.2 (A), J1.3, J1.5, J2.4 (VDD), J2.6 (VSS), J2.MP1, L_3.3_1.1, POWER_EXP_1.1 (Pin_1), POWER_EXP_1.3 (Pin_3), POWER_EXP_1.4 (Pin_4), PROG1.1 (C), R1.1, RESET1.1 (C), R_TMC_1.1, R_TMC_2.1, R_esp_1.2, R_esp_2.1, R_tmc_15.2, R_tmc_17.2, U1.4 (GND); no longer C_tmc_9.2, L3.3_1.2
- net +48V: now also C_12v_?.1, C_3.3v_?.1, C_tmc_13.1, C_tmc_14.1, C_tmc_15.1, J3.7 (Pin_7), Q5.5 (D), Q7.5 (D), R_tmc_?.2; no longer C_TMC_11.2, C_TMC_14.1, C_tmc_9.1, U_TRINAMIC1.33 (VS)
- net Reset: now also RESET1.2 (D)
- net TMC_CPI: now also U_TRINAMIC1.32 (CPI)
- net TMC_SRAH: now also C_tmc_?.1
- net TMC_SRAL: now also U_TRINAMIC1.7 (SRAL), C_tmc_?.2; no longer U_TRINAMIC1.10 (SRBL)
- net ESP_GPIO_25: now reaches U_ESP_Brain1.10 (IO25)
- net ESP_GPIO_25: now also GPIO_EXP_1.4 (Pin_4)
- net ESP_GPIO_26: now reaches U_ESP_Brain1.11 (IO26)
- net ESP_GPIO_26: now also GPIO_EXP_2.1 (Pin_1)
- net ESP_GPIO_27: now reaches U_ESP_Brain1.12 (IO27)
- net ESP_GPIO_27: now also GPIO_EXP_2.2 (Pin_2)
- net HSPI_CLK: now reaches U_ESP_Brain1.13 (IO14)
- net HSPI_CLK: now also J2.5 (CLX)
- net HSPI_MISO: now reaches U_ESP_Brain1.14 (IO12)
- net HSPI_MISO: now also J2.7 (DAT0)
- net HSPI_MOSI: now reaches U_ESP_Brain1.16 (IO13)
- net HSPI_MOSI: now also J2.3 (CMD)
- net HSPI_CS: now reaches U_ESP_Brain1.23 (IO15)
- net HSPI_CS: now also J2.2 (CD/DAT3)
- net ESP_LED: now reaches U_ESP_Brain1.24 (IO2)
- net ESP_LED: now also D1.2 (A)
- net Program: now reaches U_ESP_Brain1.25 (IO0)
- net Program: now also R_PROG_1.2, PROG1.2 (D)
- net ESP_GPIO_4: now reaches U_ESP_Brain1.26 (IO4)
- net ESP_GPIO_4: now also GPIO_EXP_1.1 (Pin_1)
- net ESP_GPIO_16: now reaches U_ESP_Brain1.27 (IO16)
- net ESP_GPIO_16: now also GPIO_EXP_1.2 (Pin_2)
- net ESP_GPIO_17: now reaches U_ESP_Brain1.28 (IO17)
- net ESP_GPIO_17: now also GPIO_EXP_1.3 (Pin_3)
- net VSPI_CS: now reaches U_ESP_Brain1.29 (IO5)
- net VSPI_CS: now also U_TRINAMIC1.13 (CSN_CFG3)
- net VSPI_CLK: now reaches U_ESP_Brain1.30 (IO18)
- net VSPI_CLK: now also U_TRINAMIC1.14 (SCK_CFG2)
- net VSPI_MISO: now reaches U_ESP_Brain1.31 (IO19)
- net VSPI_MISO: now also U_TRINAMIC1.16 (SDO_CFG0)
- net ESP_I2C_SDA: now reaches U_ESP_Brain1.33 (IO21)
- net ESP_I2C_SDA: now also C_esp_1.2, R_esp_1.1, U1.1 (SDA)
- net ESP_I2C_SCL: now reaches U_ESP_Brain1.36 (IO22)
- net ESP_I2C_SCL: now also C_esp_2.1, R_esp_2.2, U1.7 (SCL)
- net VSPI_MOSI: now reaches U_ESP_Brain1.37 (IO23)
- net VSPI_MOSI: now also U_TRINAMIC1.15 (SDI_CFG1)
- net ESP_Emergency: now reaches U_ESP_Brain1.6 (IO34)
- net ESP_Emergency: now also U_TRINAMIC1.28 (DRV_ENN), J1.4, R_TMC_1.2
- net ESP_GPIO_32: now reaches U_ESP_Brain1.8 (IO32)
- net ESP_GPIO_32: now also GPIO_EXP_2.3 (Pin_3)
- net ESP_GPIO_33: now reaches U_ESP_Brain1.9 (IO33)
- net ESP_GPIO_33: now also GPIO_EXP_2.4 (Pin_4)
- net at C_3.3v_6.1, D_3.3_1.1 (K), U_48v_to_3.3v1.5 (OUT): now also L3.3_1.2; no longer L3.3_1.1, U_48v_to_3.3v1.6 (OUT)
- net at C_12v_6.1, D_12v_1.1 (K), U_48v_to_12v1.5 (OUT): now also L12v_1.2; no longer L_12v_1.1, U_48v_to_12v1.6 (OUT)
- net TMC_HB1: now reaches U_TRINAMIC1.1 (HB1)
- net TMC_HB1: now also R_tmc_11.2
- net TMC_CB1: now reaches U_TRINAMIC1.2 (CB1)
- net TMC_CB1: now also C_tmc_10.2
- net TMC_Ramp: now reaches U_TRINAMIC1.21 (SD_MODE)
- net TMC_Ramp: now also R_TMC_2.2
- net Encoder_B: now reaches U_TRINAMIC1.23 (ENCB_DCEN_CFG4)
- net Encoder_B: now also J3.6 (Pin_6)
- net Encoder_A: now reaches U_TRINAMIC1.24 (ENCA_DCIN_CFG5)
- net Encoder_A: now also J3.5 (Pin_5)
- net Encoder_N: now reaches U_TRINAMIC1.25 (ENCN_DCO_CFG6)
- net Encoder_N: now also J3.8 (Pin_8)
- net TMC_CB2: now reaches U_TRINAMIC1.43 (CB2)
- net TMC_CB2: now also C_tmc_9.2
- net TMC_HB2: now reaches U_TRINAMIC1.44 (HB2)
- net TMC_HB2: now also R_tmc_19.1
- net TMC_BMB2: now reaches U_TRINAMIC1.45 (BMB2)
- net TMC_BMB2: now also C_tmc_9.1, D_tmc_4.1 (K), R_tmc_16.2
- net TMC_LB2: now reaches U_TRINAMIC1.46 (LB2)
- net TMC_LB2: now also R_tmc_18.1
- net TMC_LB1: now reaches U_TRINAMIC1.47 (LB1)
- net TMC_LB1: now also R_tmc_12.2
- net TMC_BMB1: now reaches U_TRINAMIC1.48 (BMB1)
- net TMC_BMB1: now also C_tmc_10.1, D_tmc_2.1 (K), R_tmc_13.2
- net TMC_SRBH: now reaches U_TRINAMIC1.9 (SRBH)
- net TMC_SRBH: now also C_tmc_11.1, R_tmc_14.1
- net at Q3.1 (S), Q3.2 (S), Q3.3 (S)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: now also C_tmc_?.1
- net Stepper_Loop_1_1 renamed Stepper_Loop_A_1
- net Stepper_Loop_A_1: now also J3.1 (Pin_1)
- net Stepper_Loop_1_2 renamed Stepper_Loop_A_2
- net Stepper_Loop_A_2: now also J3.2 (Pin_2)
- new net: D_1esp_2.1 (K), J1.1, R_esp_3.1, U1.2 (RXD-SDA), U1.3 (TXD-SDA)
- new net: D_1esp_1.1 (K), J1.8, R_esp_4.2, U1.5 (TXD-SCL), U1.6 (RXD-SCL)
- new net: Q7.4 (G), R_tmc_19.2
- new net: C_tmc_?.1, Q6.1 (S), Q6.2 (S), Q6.3 (S), Q8.1 (S), Q8.2 (S), Q8.3 (S), R_tmc_14.2, R_tmc_17.1
- new net: Q8.4 (G), R_tmc_18.2
- new net: Q6.4 (G), R_tmc_12.1
- new net: Q5.4 (G), R_tmc_11.1
- new net: D1.1 (K), R1.2
- new net: L3.3_1.1, L_3.3_1.2
- new net: L12v_1.1, L_12v_1.2
- new net Stepper_Loop_B_1: C_TMC_28.2, J3.3 (Pin_3), Q5.1 (S), Q5.2 (S), Q5.3 (S), Q6.5 (D), R_tmc_13.1
- new net Stepper_Loop_B_2: C_TMC_29.2, J3.4 (Pin_4), Q7.1 (S), Q7.2 (S), Q7.3 (S), Q8.5 (D), R_tmc_16.1
- new net TMC_SRBL: C_tmc_11.2, R_tmc_15.1, U_TRINAMIC1.10 (SRBL)
- new net TMC_VS: C_TMC_11.2, C_TMC_14.1, R_tmc_?.1, U_TRINAMIC1.33 (VS)
- no-connect marks 0 -> 24
Other:
- note added: "ESP32 / Logic"
- note added: "Emergency\nStop"
- note added: "GPIO\nEXP"
- note added: "I2C Connectors"
- note added: "LED"
- note added: "Power"
- note added: "Power EXP"
- note added: "Ramp Tie\nDown"
- note added: "SD Card Reader"
- note added: "Stepper Connector"
- note added: "Stepper Controller"
- note added: "Stepper Loop A Mosfets"
- note added: "Stepper Loop B Mosfets"
- note added: "Stepper Mgmt."
- note removed: "Stepper Loop 1 Mosfets"
- moved on the sheet: C3, C4, C_12_4, C_12v_1, C_12v_2, C_12v_4, C_12v_6, C_12v_8, C_3.3_2, C_3.3_4, C_3.3v_1, C_3.3v_4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
