File: hardware/electronics/main_board/main_board_cheaper.kicad_pcb (KiCad board)
At the start: 2 copper layers, 125.5 x 125.5 mm, 147 parts, among them J1 RJ45, J2 TF-15X15, J3 Conn_02x04_Odd_Even, Q1 CSD18537NQ5A, Q2 CSD18537NQ5A, Q3 CSD18537NQ5A, Q4 CSD18537NQ5A, Q5 CSD18537NQ5A, Q6 CSD18537NQ5A, Q7 CSD18537NQ5A, Q8 CSD18537NQ5A, U1 P82B96

Commit message: fixed pcb issues - still untested
Parts:
- added REF**: OSHW-Logo2_7.3x6mm_Copper, Symbol:OSHW-Logo2_7.3x6mm_Copper, F.Cu at (134.0, 98.5)
- added REF**: KiCad-Logo_6mm_Copper, Symbol:KiCad-Logo_6mm_Copper, F.Cu at (133.5, 123.0)
- J1: footprint main_board:2158771 -> main_board:5555166-1
- moved J1 17.5 mm to (13.1, 14.1), turned to 180 degrees
Routing:
- net Net-(D_esp_2-Pad1): track 47.7 -> 66.9 mm, vias 0 -> 1
- net ESP_Emergency: track 123.7 -> 133.0 mm
- net 3.3_comp_cap1: track 398.4 -> 404.4 mm, vias 6 -> 8
- net 12v_comp_cap1: track 325.1 -> 329.9 mm
- net Net-(D_esp_1-Pad1): track 61.6 -> 66.0 mm
- net TMC_CPI: track 97.0 -> 98.9 mm
- net TMC_5VOUT: track 20.7 -> 22.3 mm
- net 12v_comp_cap2: track 1425.9 -> 1427.3 mm, vias 56 -> 51
- net TMC_VS: track 32.5 -> 33.7 mm
- net TMC_CB1: track 38.0 -> 38.6 mm
Other:
- board text added: "48v In"
- board text added: "<1A Power Exp"
- board text added: "AutoPen v2 Prototype #1"
- board text added: "ESP GPIO EXP"
- board text added: "PROG"
- board text added: "Prog Headers"
- board text added: "RESET"
- board text added: "Stepper Connector"
