File: hardware/electronics/main_board/main_board_cheaper.sch (KiCad schematic (older format))
At the start: 144 parts, among them J1 RJ45, J2 TF-15X15, J3 Conn_02x04_Odd_Even, Q1 CSD18537NQ5A, Q2 CSD18537NQ5A, Q3 CSD18537NQ5A, Q4 CSD18537NQ5A, Q5 CSD18537NQ5A, Q6 CSD18537NQ5A, Q7 CSD18537NQ5A, Q8 CSD18537NQ5A, U1 P82B96

Commit message: fixed pcb issues - still untested
Parts:
- J1: footprint main_board:2158771 -> main_board:5555166-1; JLCPCB C305919 -> C305991
- U_TRINAMIC1: JLCPCB (none) -> C516354
Changed lines of the file:
@@
 F 11 "Trinamic Motion Control GmbH" H 15700 9700 60  0001 L CNN "Manufacturer"
 F 12 "Active" H 15700 9800 60  0001 L CNN "Status"
+F 13 "C516354" H 14850 8600 50  0001 C CNN "JLCPCB"
 	1    14850 8600
 	1    0    0    -1
@@
 F 0 "J1" H 9150 4225 50  0000 R CNN
 F 1 "RJ45" H 9200 4300 50  0000 R CNN
-F 2 "main_board:2158771" V 9150 4775 50  0001 C CNN
+F 2 "main_board:5555166-1" V 9150 4775 50  0001 C CNN
 F 3 "~" V 9150 4775 50  0001 C CNN
-F 4 "C305919" H 9150 4750 50  0001 C CNN "JLCPCB"
+F 4 "C305991" H 9150 4750 50  0001 C CNN "JLCPCB"
 	1    9150 4750
 	-1   0    0    1
