File: hardware/electronics/main_board/main_board_cheaper2.sch (KiCad schematic (older format))
At the start: 144 parts, among them J1 TF-15X15, J2 RJ45, J3 Conn_02x04_Odd_Even, Q1 CSD18537NQ5A, Q2 CSD18537NQ5A, Q3 CSD18537NQ5A, Q4 CSD18537NQ5A, Q5 CSD18537NQ5A, Q6 CSD18537NQ5A, Q7 CSD18537NQ5A, Q8 CSD18537NQ5A, U1 P82B96

Commit message: updated footprint to generic SOIC-16w so tooling rotates it properly."
Parts:
- U_48v_to_12v1, U_48v_to_3.3v1: footprint main_board:SOIC127P1032X265-16N -> Package_SO:SOIC-16W_7.5x10.3mm_P1.27mm
Changed lines of the file:
@@
 F 0 "U_48v_to_3.3v1" H 12700 4050 79  0000 C CNN
 F 1 "L4978D" H 12700 3950 79  0000 C CNN
-F 2 "main_board:SOIC127P1032X265-16N" H 12700 3600 79  0001 C CNN
+F 2 "Package_SO:SOIC-16W_7.5x10.3mm_P1.27mm" H 12700 3600 79  0001 C CNN
 F 3 "https://datasheet.lcsc.com/szlcsc/1809291616_STMicroelectronics-L4978D_C93521.pdf" H 12700 3600 79  0001 C CNN
 F 4 "C93521" H 12700 3600 50  0001 C CNN "JLCPCB"
@@
 F 0 "U_48v_to_12v1" H 12200 1975 79  0000 C CNN
 F 1 "L4978D" H 12200 1875 79  0000 C CNN
-F 2 "main_board:SOIC127P1032X265-16N" H 12200 1525 79  0001 C CNN
+F 2 "Package_SO:SOIC-16W_7.5x10.3mm_P1.27mm" H 12200 1525 79  0001 C CNN
 F 3 "https://datasheet.lcsc.com/szlcsc/1809291616_STMicroelectronics-L4978D_C93521.pdf" H 12200 1525 79  0001 C CNN
 F 4 "C93521" H 12200 1525 50  0001 C CNN "JLCPCB"

Commit message: added power split pcb
Parts:
- C_12v_7, C_3.3v_8: footprint Capacitor_SMD:C_0805_2012Metric -> Capacitor_SMD:C_0603_1608Metric
- C_TMC_26: footprint Capacitor_SMD:C_1206_3216Metric -> Capacitor_SMD:C_0805_2012Metric
- J3: JLCPCB C239456 -> C277661
Changed lines of the file:
@@
 F 0 "C_TMC_26" H 4367 8246 50  0000 L CNN
 F 1 "470nF" H 4367 8155 50  0000 L CNN
-F 2 "Capacitor_SMD:C_1206_3216Metric" H 4275 8200 50  0001 C CNN
+F 2 "Capacitor_SMD:C_0805_2012Metric" H 4275 8200 50  0001 C CNN
 F 3 "~" H 4275 8200 50  0001 C CNN
 F 4 "C13967" H 4275 8200 50  0001 C CNN "JLCPCB"
@@
 F 2 "Connector_Molex:Molex_Micro-Fit_3.0_43045-0812_2x04_P3.00mm_Vertical" H 12725 9400 50  0001 C CNN
 F 3 "~" H 12725 9400 50  0001 C CNN
-F 4 "C239456" H 12725 9400 50  0001 C CNN "JLCPCB"
+F 4 "C277661" H 12725 9400 50  0001 C CNN "JLCPCB"
 	1    12725 9400
 	1    0    0    -1
@@
 F 0 "C_12v_7" V 15300 2200 50  0000 L CNN
 F 1 "68nF" V 15375 2200 50  0000 L CNN
-F 2 "Capacitor_SMD:C_0805_2012Metric" H 15350 2050 50  0001 C CNN
+F 2 "Capacitor_SMD:C_0603_1608Metric" H 15350 2050 50  0001 C CNN
 F 3 "~" H 15350 2050 50  0001 C CNN
 F 4 "C31658" V 15350 2050 50  0001 C CNN "JLCPCB"
@@
 F 0 "C_3.3v_8" V 15500 4275 50  0000 L CNN
 F 1 "68nF" V 15575 4275 50  0000 L CNN
-F 2 "Capacitor_SMD:C_0805_2012Metric" H 15550 4125 50  0001 C CNN
+F 2 "Capacitor_SMD:C_0603_1608Metric" H 15550 4125 50  0001 C CNN
 F 3 "~" H 15550 4125 50  0001 C CNN
 F 4 "C31658" V 15550 4125 50  0001 C CNN "JLCPCB"
